File: StreamDeck/Subcircuito_comunicação.sch (KiCad schematic (older format))
At the start: 11 parts, among them J1 USB_B_Micro, J2 sd_CARD_READER_MODULE, U3 CH340G, Y1 12MHz

Commit message: Schematic_v1.1
Esquematico usando um Atmega48v para controlar e fazer um stream deck.
Parts:
- added C15: c, symbol Device:C
- added D2, D3: LED, symbol Device:LED
- added R20, R21, R22: 1K, symbol Device:R
- R1: value 4k7 -> 1K
- renumbered J2 to J10, J1 to J11
Connections:
- net +5V: now also R22.1
- net RXD: now also D3.1 (K), R21.1; no longer R1.2, U3.3 (RXD)
- net TXD: now also D2.1 (K), R20.1; no longer U3.2 (TXD)
- net at U3.13 (~DTR): now also C15.2
- new net: R20.2, U3.2 (TXD)
- new net: R21.2, U3.3 (RXD)
- new net: D3.2 (A), R1.2
- new net: D2.2 (A), R22.2
- new net RST_ARDUINO: C15.1
- no-connect marks 8 -> 7
Other:
- moved on the sheet: R1
Changed lines of the file:
@@
 P 5950 6400
 AR Path="/5FF4D7B1" Ref="J?"  Part="1"
-AR Path="/5FF3D484/5FF4D7B1" Ref="J2"  Part="1"
-F 0 "J2" H 5978 6376 50  0000 L CNN
+AR Path="/5FF3D484/5FF4D7B1" Ref="J10"  Part="1"
+F 0 "J10" H 5978 6376 50  0000 L CNN
 F 1 "sd_CARD_READER_MODULE" H 5978 6285 50  0000 L CNN
 F 2 "" H 5950 6400 50  0001 C CNN
@@
 $EndComp
 $Comp
-L Connector:USB_B_Micro J1
+L Connector:USB_B_Micro J11
 U 1 1 5FF6F5F8
 P 3200 3750
-F 0 "J1" H 3257 4217 50  0000 C CNN
+F 0 "J11" H 3257 4217 50  0000 C CNN
 F 1 "USB_B_Micro" H 3257 4126 50  0000 C CNN
 F 2 "" H 3350 3700 50  0001 C CNN
@@
 	1    0    0    -1
 $EndComp
-Text GLabel 6100 3300 2    50   Input ~ 0
+Text GLabel 7450 3300 2    50   Input ~ 0
 TXD
-Text GLabel 6500 3250 1    50   Input ~ 0
+Text GLabel 7450 3400 2    50   Input ~ 0
 RXD
 $Comp
@@
 L Device:R R1
 U 1 1 5FF762E4
-P 6700 3150
-F 0 "R1" H 6770 3196 50  0000 L CNN
-F 1 "4k7" H 6770 3105 50  0000 L CNN
-F 2 "" V 6630 3150 50  0001 C CNN
-F 3 "~" H 6700 3150 50  0001 C CNN
-	1    6700 3150
-	1    0    0    -1
-$EndComp
-Wire Wire Line
-	6700 3300 6700 3400
-Wire Wire Line
-	6100 3400 6500 3400
+P 6900 2850
+F 0 "R1" H 6970 2896 50  0000 L CNN
+F 1 "1K" H 6970 2805 50  0000 L CNN
+F 2 "" V 6830 2850 50  0001 C CNN
+F 3 "~" H 6900 2850 50  0001 C CNN
+	1    6900 2850
+	1    0    0    -1
+$EndComp
+Wire Wire Line
+	6900 3000 6900 3100
 $Comp
 L power:+5V #PWR06
@@
 L power:+5V #PWR09
 U 1 1 5FF777B5
-P 6700 2900
-F 0 "#PWR09" H 6700 2750 50  0001 C CNN
-F 1 "+5V" H 6715 3073 50  0000 C CNN
-F 2 "" H 6700 2900 50  0001 C CNN
-F 3 "" H 6700 2900 50  0001 C CNN
-	1    6700 2900
-	1    0    0    -1
-$EndComp
-Wire Wire Line
-	6700 2900 6700 3000
-Wire Wire Line
-	6500 3250 6500 3400
-Connection ~ 6500 3400
-Wire Wire Line
-	6500 3400 6700 3400
+P 6900 2600
+F 0 "#PWR09" H 6900 2450 50  0001 C CNN
+F 1 "+5V" H 6915 2773 50  0000 C CNN
+F 2 "" H 6900 2600 50  0001 C CNN
+F 3 "" H 6900 2600 50  0001 C CNN
+	1    6900 2600
+	1    0    0    -1
+$EndComp
+Wire Wire Line
+	6900 2600 6900 2700
 $Comp
 L Device:C C14
@@
 NoConn ~ 6100 3800
 NoConn ~ 6100 3900
-NoConn ~ 6100 4000
 NoConn ~ 6100 4100
+Text GLabel 6900 4000 2    50   Input ~ 0
+RST_ARDUINO
+$Comp
+L Device:C C15
+U 1 1 5FF951A8
+P 6450 4000
+F 0 "C15" V 6198 4000 50  0000 C CNN
+F 1 "c" V 6289 4000 50  0000 C CNN
+F 2 "" H 6488 3850 50  0001 C CNN
+F 3 "~" H 6450 4000 50  0001 C CNN
+	1    6450 4000
+	0    1    1    0
+$EndComp
+Wire Wire Line
+	6600 4000 6900 4000
+Wire Wire Line
+	6300 4000 6100 4000
+$Comp
+L Device:LED D3
+U 1 1 5FF9F39B
+P 6900 3250
+F 0 "D3" V 6939 3132 50  0000 R CNN
+F 1 "LED" V 6848 3132 50  0000 R CNN
+F 2 "" H 6900 3250 50  0001 C CNN
+F 3 "~" H 6900 3250 50  0001 C CNN
+	1    6900 3250
+	0    -1   -1   0
+$EndComp
+$Comp
+L Device:R R22
+U 1 1 5FFA2664
+P 6650 2750
+F 0 "R22" H 6720 2796 50  0000 L CNN
+F 1 "1K" H 6720 2705 50  0000 L CNN
+F 2 "" V 6580 2750 50  0001 C CNN
+F 3 "~" H 6650 2750 50  0001 C CNN
+	1    6650 2750
+	1    0    0    -1
+$EndComp
+Wire Wire Line
+	6650 2900 6650 3000
+$Comp
+L power:+5V #PWR055
+U 1 1 5FFA266B
+P 6650 2500
+F 0 "#PWR055" H 6650 2350 50  0001 C CNN
+F 1 "+5V" H 6665 2673 50  0000 C CNN
+F 2 "" H 6650 2500 50  0001 C CNN
+F 3 "" H 6650 2500 50  0001 C CNN
+	1    6650 2500
+	1    0    0    -1
+$EndComp
+Wire Wire Line
+	6650 2500 6650 2600
+$Comp
+L Device:LED D2
+U 1 1 5FFA2672
+P 6650 3150
+F 0 "D2" V 6689 3032 50  0000 R CNN
+F 1 "LED" V 6598 3032 50  0000 R CNN
+F 2 "" H 6650 3150 50  0001 C CNN
+F 3 "~" H 6650 3150 50  0001 C CNN
+	1    6650 3150
+	0    -1   -1   0
+$EndComp
+$Comp
+L Device:R R20
+U 1 1 5FFA3205
+P 6350 3300
+F 0 "R20" V 6143 3300 50  0000 C CNN
+F 1 "1K" V 6234 3300 50  0000 C CNN
+F 2 "" V 6280 3300 50  0001 C CNN
+F 3 "~" H 6350 3300 50  0001 C CNN
+	1    6350 3300
+	0    1    1    0
+$EndComp
+$Comp
+L Device:R R21
+U 1 1 5FFA3860
+P 6550 3400
+F 0 "R21" V 6650 3250 50  0000 C CNN
+F 1 "1K" V 6650 3400 50  0000 C CNN
+F 2 "" V 6480 3400 50  0001 C CNN
+F 3 "~" H 6550 3400 50  0001 C CNN
+	1    6550 3400
+	0    1    1    0
+$EndComp
+Wire Wire Line
+	6200 3300 6100 3300
+Wire Wire Line
+	6650 3300 6500 3300
+Wire Wire Line
+	6900 3400 6700 3400
+Wire Wire Line
+	6400 3400 6100 3400
+Wire Wire Line
+	6650 3300 7450 3300
+Connection ~ 6650 3300
+Wire Wire Line
+	6900 3400 7450 3400
+Connection ~ 6900 3400
 $EndSCHEMATC
